Commit message: Forklift navigation significantly better as tested in the depot world.

File: urdf/RX20_16/front_wheels.xacro (robot description, xacro)
@@ -24,5 +24,5 @@
     <parent link="base_link" />
     <child link="wheel_${name}_driving_link" />
-    <origin xyz="${x_loading} ${y_loading} ${z_loading}" rpy="1.57 0 0" />
+    <origin xyz="${x_loading} ${y_loading} ${z_loading}" rpy="1.570796 0 0" />
     <axis xyz="0 0 ${1*flip}" />
     <!-- <joint_properties damping="1.0" friction="1.0"/> -->

File: urdf/RX20_16/main.xacro (robot description, xacro)
@@ -18,6 +18,6 @@
 <!-- <xacro:detection_lidar name="front"  x="0.0"  y="0.0" z="2.0" roll="0" pitch="0" yaw="0" resolution="1"/> -->
 <!-- <xacro:nav_lidar name="back"  x="-1.65"  y="0.0" z="0.0" roll="0" pitch="0" yaw="3.14509" resolution="1"/> -->
-<xacro:nav_lidar name="rf"  x="0.3"  y="-0.6" z="0.0" roll="0" pitch="0" yaw="-1.57" resolution="1"/>
-<xacro:nav_lidar name="lf"  x="0.3"  y="+0.6" z="0.0" roll="0" pitch="0" yaw="+1.57" resolution="1"/>
+<xacro:nav_lidar name="rf"  x="0.3"  y="-0.6" z="0.0" roll="0" pitch="0" yaw="-1.570796" resolution="1"/>
+<xacro:nav_lidar name="lf"  x="0.3"  y="+0.6" z="0.0" roll="0" pitch="0" yaw="+1.570796" resolution="1"/>
 <!-- <xacro:detection_lidar name="front"  x="0.0"  y="0.0" z="0.6" roll="0" pitch="0" yaw="0" resolution="1"/> -->
 </robot>

File: urdf/RX20_16/nav_lidar.xacro (robot description, xacro)
@@ -32,8 +32,8 @@
   <gazebo reference="${name}_nav_lidar">
       <sensor name="${name}_nav_lidar" type="gpu_lidar">
-      <static>false</static>
+      <!-- <static>false</static> -->
       <always_on>true</always_on>
       <visualize>true</visualize>
-      <pose>0 0 0 0 0 0</pose>
+      <!-- <pose>0 0 0 0 0 0</pose> -->
       <update_rate>10</update_rate>
       <topic>/lidar_${name}/scan</topic>
@@ -44,6 +44,6 @@
             <samples>360</samples>
             <resolution>1.000000</resolution>
-            <min_angle>-1.5708</min_angle>
-            <max_angle>1.5708</max_angle>
+            <min_angle>-1.570796</min_angle>
+            <max_angle>1.570796</max_angle>
           </horizontal>
         </scan>

File: urdf/RX20_16/steer_wheels.xacro (robot description, xacro)
@@ -24,5 +24,5 @@
     <parent link="base_link" />
     <child link="wheel_${name}_steering_link" />
-    <origin xyz="${x_steering} ${y_steering} ${z_steering }" rpy="0 0 1.57" />
+    <origin xyz="${x_steering} ${y_steering} ${z_steering }" rpy="0 0 1.570796" />
     <!-- <origin xyz="-0.662 0.247 0.115" rpy="0 0 0" /> -->
     <axis xyz="0 0 ${1*flip}" />
@@ -53,5 +53,5 @@
     <parent link="wheel_${name}_steering_link" />
     <child link="wheel_${name}_link" />
-    <origin xyz=" 0 0 -0.09" rpy="0 1.57 0" />
+    <origin xyz=" 0 0 -0.09" rpy="0 1.570796 0" />
     <axis xyz="0 0 1" />
     <!-- <joint_properties damping="1.0" friction="0.3"/> -->

File: urdf/RX20_16/wheel_control.xacro (robot description, xacro)
@@ -5,5 +5,5 @@
         filename="gz-sim-diff-drive-system"
         name="gz::sim::systems::DiffDrive">
-        <wheel_separation>1.12</wheel_separation>
+        <wheel_separation>0.932</wheel_separation>
         <wheel_radius>0.18</wheel_radius>
         <update_rate>30</update_rate>
@@ -11,5 +11,13 @@
         <right_joint>wheel_right_driving_joint</right_joint>
         <max_wheel_torque>200</max_wheel_torque>
-        <max_wheel_acceleration>1</max_wheel_acceleration>
+        <!-- <max_wheel_acceleration>0.1</max_wheel_acceleration> -->
+        <max_linear_acceleration>0.5</max_linear_acceleration>
+        <min_linear_acceleration>-0.5</min_linear_acceleration>
+        <max_angular_acceleration>0.5</max_angular_acceleration>
+        <min_angular_acceleration>-0.5</min_angular_acceleration>
+        <max_linear_velocity>0.5</max_linear_velocity>
+        <min_linear_velocity>-0.5</min_linear_velocity>
+        <max_angular_velocity>0.3</max_angular_velocity>
+        <min_angular_velocity>-0.3</min_angular_velocity>
         <topic>/cmd_vel</topic>
         <odom_topic>/odom</odom_topic>
