Commit message: Fixed dae loading so RViz would render the forklift.

File: urdf/RX20_16/base.xacro (robot description, xacro)
@@ -12,5 +12,5 @@
       <origin rpy="0 0 0" xyz="0 0 0"/>
       <geometry>
-        <mesh filename="$(find wb_nav2_bringup)/urdf/RX20_16/meshes/body.dae" />
+        <mesh filename="file:$(find wb_nav2_bringup)/urdf/RX20_16/meshes/body.dae" />
       </geometry>
     </collision>
@@ -18,5 +18,5 @@
       <origin rpy="0 0 0" xyz="0 0 0"/>
       <geometry>
-        <mesh filename="$(find wb_nav2_bringup)/urdf/RX20_16/meshes/body.dae" />
+        <mesh filename="file:$(find wb_nav2_bringup)/urdf/RX20_16/meshes/body.dae" />
       </geometry>
     </visual>

File: urdf/RX20_16/front_wheels.xacro (robot description, xacro)
@@ -17,5 +17,5 @@
     <origin xyz="0 0 0" rpy="0 0 0"/>
     <geometry>
-        <mesh filename="$(find wb_nav2_bringup)/urdf/RX20_16/meshes/front_wheel.dae" />
+        <mesh filename="file:$(find wb_nav2_bringup)/urdf/RX20_16/meshes/front_wheel.dae" />
     </geometry>
     </visual>

File: urdf/RX20_16/loading_forklift_joints.xacro (robot description, xacro)
@@ -9,5 +9,5 @@
     <collision >
     <origin xyz="0 0 0" rpy="0 0 0"/>
-    <geometry> <mesh filename="$(find wb_nav2_bringup)/urdf/RX20_16/meshes/tilt_link.dae" />
+    <geometry> <mesh filename="file:$(find wb_nav2_bringup)/urdf/RX20_16/meshes/tilt_link.dae" />
     </geometry>
     </collision>
@@ -15,5 +15,5 @@
     <origin xyz="0 0 0" rpy="0 0 0"/>
     <geometry>
-          <mesh filename="$(find wb_nav2_bringup)/urdf/RX20_16/meshes/tilt_link.dae" />
+          <mesh filename="file:$(find wb_nav2_bringup)/urdf/RX20_16/meshes/tilt_link.dae" />
     </geometry>
     </visual>
@@ -36,5 +36,5 @@
     <collision >
     <origin xyz="0 0 0" rpy="0 0 0"/>
-    <geometry> <mesh filename="$(find wb_nav2_bringup)/urdf/RX20_16/meshes/lift_link.dae" />
+    <geometry> <mesh filename="file:$(find wb_nav2_bringup)/urdf/RX20_16/meshes/lift_link.dae" />
     </geometry>
     </collision>
@@ -42,5 +42,5 @@
     <origin xyz="0 0 0" rpy="0 0 0"/>
     <geometry>
-          <mesh filename="$(find wb_nav2_bringup)/urdf/RX20_16/meshes/lift_link.dae" />
+          <mesh filename="file:$(find wb_nav2_bringup)/urdf/RX20_16/meshes/lift_link.dae" />
     </geometry>
     </visual>
@@ -63,5 +63,5 @@
     <collision >
     <origin xyz="0 0 0" rpy="0 0 0"/>
-    <geometry> <mesh filename="$(find wb_nav2_bringup)/urdf/RX20_16/meshes/sideshift_link.dae" />
+    <geometry> <mesh filename="file:$(find wb_nav2_bringup)/urdf/RX20_16/meshes/sideshift_link.dae" />
     </geometry>
     </collision>
@@ -69,5 +69,5 @@
     <origin xyz="0 0 0" rpy="0 0 0"/>
     <geometry>
-          <mesh filename="$(find wb_nav2_bringup)/urdf/RX20_16/meshes/sideshift_link.dae" />
+          <mesh filename="file:$(find wb_nav2_bringup)/urdf/RX20_16/meshes/sideshift_link.dae" />
     </geometry>
     </visual>

File: urdf/RX20_16/steer_wheels.xacro (robot description, xacro)
@@ -9,20 +9,20 @@
     </inertial>
     <collision >
-    <origin xyz="0 0 0" rpy="0 0 0"/>
-    <geometry>
-        <mesh filename="$(find wb_nav2_bringup)/urdf/RX20_16/meshes/steering_rod.dae" />
-    </geometry>
+      <origin xyz="0 0 0" rpy="0 0 0"/>
+      <geometry>
+          <mesh filename="file:$(find wb_nav2_bringup)/urdf/RX20_16/meshes/steering_rod.dae" />
+      </geometry>
     </collision>
     <visual >
-    <origin xyz="0 0 0" rpy="0 0 0"/>
-    <geometry>
-        <mesh filename="$(find wb_nav2_bringup)/urdf/RX20_16/meshes/steering_rod.dae" />
-    </geometry>
+      <origin xyz="0 0 0" rpy="0 0 0"/>
+      <geometry>
+          <mesh filename="file:$(find wb_nav2_bringup)/urdf/RX20_16/meshes/steering_rod.dae" />
+      </geometry>
     </visual>
   </link>
-  <joint name="wheel_${name}_steering_joint" type="revolute">
+  <joint name="wheel_${name}_steering_joint" type="fixed">
     <parent link="base_link" />
     <child link="wheel_${name}_steering_link" />
-    <origin xyz="${x_steering} ${y_steering} ${z_steering }" rpy="0 0 1.570796" />
+    <origin xyz="${x_steering} ${y_steering} ${z_steering}" rpy="0 0 1.570796" />
     <!-- <origin xyz="-0.662 0.247 0.115" rpy="0 0 0" /> -->
     <axis xyz="0 0 ${1*flip}" />
@@ -46,9 +46,9 @@
     <origin xyz="0 0 0" rpy="0 0 0"/>
     <geometry>
-        <mesh filename="$(find wb_nav2_bringup)/urdf/RX20_16/meshes/rear_wheel.dae" />
+        <mesh filename="file:$(find wb_nav2_bringup)/urdf/RX20_16/meshes/rear_wheel.dae" />
     </geometry>
     </visual>
   </link>
-  <joint name="wheel_${name}_joint" type="continuous">
+  <joint name="wheel_${name}_joint" type="fixed">
     <parent link="wheel_${name}_steering_link" />
     <child link="wheel_${name}_link" />

Commit message: Able to get to docking position, sideways pallet, and automatically stop forklift.

File: urdf/RX20_16/base.xacro (robot description, xacro)
@@ -6,6 +6,6 @@
     <inertial>
       <origin xyz="-0.8 0 0.417" rpy="0 0 0"/>
-      <xacro:box_inertia mass="10" x="1.843" y="1.1" z="0.835"/>
-      <mass value= "10"/>
+      <xacro:box_inertia mass="500" x="1.843" y="1.1" z="0.835"/>
+      <mass value= "500"/>
     </inertial>
     <collision>

File: urdf/RX20_16/camera.xacro (robot description, xacro)
@@ -39,8 +39,8 @@
       <always_on>1</always_on>
       <camera>
-        <horizontal_fov>1.25</horizontal_fov>
+        <horizontal_fov>1.0</horizontal_fov>
         <image>
-          <width>640</width>
-          <height>480</height>
+          <width>800</width>
+          <height>600</height>
         </image>
         <clip>

File: urdf/RX20_16/front_wheels.xacro (robot description, xacro)
@@ -45,7 +45,7 @@
 			<!-- <kp>10000000.0</kp> -->
 			<kp>1000000000.0</kp>
-			<kd>1000.0</kd>
-			<minDepth>0.002</minDepth>
-			<maxVel>0</maxVel>
+			<kd>10.0</kd>
+			<min_depth>0.01</min_depth>
+			<max_vel>1.0</max_vel>
 		</gazebo>
  </xacro:macro>

File: urdf/RX20_16/main.xacro (robot description, xacro)
@@ -13,7 +13,7 @@
 <xacro:rx20_steer_wheel name="left" x_steering="-1.429" y_steering="0.404" z_steering="0.06" radius="0.150" width="0.15" flip="-1" />
 <xacro:rx20_steer_wheel name="right" x_steering="-1.429" y_steering="-0.404" z_steering="0.06" radius="0.150" width="0.15" flip="-1" />
-<xacro:rx20_front_wheel name="right" x_loading="0.0" y_loading="-0.466" z_loading="0.0" radius="0.18" width="0.18" flip="-1" />
-<xacro:rx20_front_wheel name="left" x_loading="0.0" y_loading="0.466" z_loading="0.0" radius="0.18" width="0.18" flip="-1" />
-<xacro:camera name="front"  x="0.4"  y="0" z="0.3" roll="0.0" pitch="0.0" yaw="0.0"/>
+<xacro:rx20_front_wheel name="right" x_loading="0.0" y_loading="-0.466" z_loading="0.0" radius="0.181" width="0.18" flip="-1" />
+<xacro:rx20_front_wheel name="left" x_loading="0.0" y_loading="0.466" z_loading="0.0" radius="0.181" width="0.18" flip="-1" />
+<xacro:camera name="front"  x="0.4"  y="0" z="0.2" roll="0.0" pitch="0.0" yaw="0.0"/>
 <!-- <xacro:nav_lidar name="top"  x="0."  y="0.0" z="2" roll="0" pitch="0" yaw="0.0" resolution="1"/> -->
 <!-- <xacro:detection_lidar name="front"  x="0.0"  y="0.0" z="2.0" roll="0" pitch="0" yaw="0" resolution="1"/> -->

File: urdf/RX20_16/wheel_control.xacro (robot description, xacro)
@@ -6,9 +6,9 @@
         name="gz::sim::systems::DiffDrive">
         <wheel_separation>0.932</wheel_separation>
-        <wheel_radius>0.18</wheel_radius>
+        <wheel_radius>0.181</wheel_radius>
         <update_rate>30</update_rate>
         <left_joint>wheel_left_driving_joint</left_joint>
         <right_joint>wheel_right_driving_joint</right_joint>
-        <max_wheel_torque>200</max_wheel_torque>
+        <max_wheel_torque>10</max_wheel_torque>
         <!-- <max_wheel_acceleration>0.1</max_wheel_acceleration> -->
         <max_linear_acceleration>0.5</max_linear_acceleration>
