Commit message: Front RGBD camera works.

File: urdf/RX20_16/camera.xacro (robot description, xacro)
@@ -1,5 +1,5 @@
 <?xml version="1.0" ?>
 <robot name="RX20_16" xmlns:xacro="http://www.ros.org/wiki/xacro">
-<xacro:macro name="camera_custom" params="name x y z roll pitch yaw ">
+<xacro:macro name="camera" params="name x y z roll pitch yaw ">
   <link name="${name}_camera_frame">
       <inertial>
@@ -11,68 +11,50 @@
       <origin xyz="0 0 0" rpy="0 0 0"/>
       <geometry>
-       <box size="0.01 0.01 0.01"/>
+       <box size="0.1 0.1 0.1"/>
       </geometry>
+      <material name="red">
+        <color rgba="1 0 0 1.0"/>
+      </material>
       </visual>
   </link>
   <joint name="${name}_camera_joint" type="fixed">
-      <parent link="base_link" />
+    <parent link="base_link" />
     <child link="${name}_camera_frame" />
     <origin xyz="${x} ${y} ${z}" rpy="${roll} ${pitch} ${yaw}" />
     <axis xyz="0 0 1" />
   </joint>
-  <link name="camera_rgbd_frame"/>
-    <joint name="camera_frame_joint" type="fixed">
-        <origin rpy="-1.5707 0 -1.5707" xyz="0 0 0"/>
-        <parent link="${name}_camera_frame"/>
-        <child link="camera_rgbd_frame"/>
-    </joint>
+    <!-- Gazebo links and joints -->
   <gazebo reference="${name}_camera_frame">
-    <sensor name="${name}_camera_frame"   type="depth">
-        <update_rate>25</update_rate>
-        <visualize>false</visualize>
-        <camera>
-            <!-- <vertical_fov>0.7</vertical_fov> unsupported -->
-          <horizontal_fov>1.047</horizontal_fov>
-            <image>
-            <format>R8G8B8</format>
-            <width>352</width>
-              <height>264</height>
-          </image>
-          <clip>
-            <near>0.3</near>
-              <far>10</far>
-          </clip>
-          <noise>
-            <type>gaussian</type>
-              <mean>0.0</mean>
-            <stddev>0.02</stddev>
-          </noise>
-          </camera>
-        <plugin filename="libgazebo_ros_openni_kinect.so" name="camera_plugin">
-          <baseline>0.2</baseline>
-          <alwaysOn>true</alwaysOn>
-            <!-- Keep this zero, update_rate in the parent <sensor> tag
-                will control the frame rate. -->
-          <updateRate>0.0</updateRate>
-            <cameraName>${name}_camera_frame</cameraName>
-          <imageTopicName>/${name}_camera_frame/depth/image_raw</imageTopicName>
-            <cameraInfoTopicName>/${name}_camera_frame/depth/camera_info</cameraInfoTopicName>
-            <depthImageTopicName>/${name}_camera_frame/depth/image_raw</depthImageTopicName>
-            <depthImageInfoTopicName>/${name}_camera_frame/depth/camera_info</depthImageInfoTopicName>
-            <pointCloudTopicName>/${name}_camera_frame/depth/points</pointCloudTopicName>
-            <frameName>camera_rgbd_frame</frameName>
-          <pointCloudCutoff>0.05</pointCloudCutoff>
-            <distortionK1>1</distortionK1>
-          <distortionK2>1</distortionK2>
-            <distortionK3>1</distortionK3>
-          <distortionT1>1</distortionT1>
-            <distortionT2>1</distortionT2>
-          <CxPrime>0</CxPrime>
-          <Cx>0</Cx>
-            <Cy>0</Cy>
-          <focalLength>0</focalLength>
-          <hackBaseline>0</hackBaseline>
-          </plugin>
-      </sensor>
+    <sensor name="rgbd_camera" type="rgbd_camera">
+      <always_on>1</always_on>
+      <camera>
+        <horizontal_fov>1.25</horizontal_fov>
+        <image>
+          <width>320</width>
+          <height>240</height>
+        </image>
+        <clip>
+          <near>0.3</near>
+          <far>100</far>
+        </clip>
+        <optical_frame_id>${name}_camera_frame</optical_frame_id>
+      </camera>
+      <update_rate>10</update_rate>
+      <visualize>true</visualize>
+      <topic>depth_camera</topic>
+      <baseline>0.2</baseline>
+      <pointCloudCutoff>0.5</pointCloudCutoff>
+      <pointCloudCutoffMax>3.0</pointCloudCutoffMax>
+      <distortionK1>0</distortionK1>
+      <distortionK2>0</distortionK2>
+      <distortionK3>0</distortionK3>
+      <distortionT1>0</distortionT1>
+      <distortionT2>0</distortionT2>
+      <CxPrime>0</CxPrime>
+      <Cx>0</Cx>
+      <Cy>0</Cy>
+      <focalLength>0</focalLength>
+      <hackBaseline>0</hackBaseline>
+    </sensor>
   </gazebo>
 </xacro:macro>

File: urdf/RX20_16/main.xacro (robot description, xacro)
@@ -4,16 +4,17 @@
 <xacro:include filename="$(find wb_nav2_bringup)/urdf/RX20_16/base.xacro" />
 <xacro:include filename="$(find wb_nav2_bringup)/urdf/RX20_16/nav_lidar.xacro" />
-<xacro:include filename="$(find wb_nav2_bringup)/urdf/RX20_16/detection_lidar.xacro" />
+<!-- <xacro:include filename="$(find wb_nav2_bringup)/urdf/RX20_16/detection_lidar.xacro" /> -->
 <xacro:include filename="$(find wb_nav2_bringup)/urdf/RX20_16/steer_wheels.xacro" />
 <xacro:include filename="$(find wb_nav2_bringup)/urdf/RX20_16/front_wheels.xacro" />
 <!-- <xacro:include filename="$(find wb_nav2_bringup)/urdf/RX20_16/d435_camera.xacro" /> -->
+<xacro:include filename="$(find wb_nav2_bringup)/urdf/RX20_16/camera.xacro" />
 <xacro:include filename="$(find wb_nav2_bringup)/urdf/RX20_16/loading_forklift_joints.xacro" />
 <xacro:include filename="$(find wb_nav2_bringup)/urdf/RX20_16/wheel_control.xacro" />
-<!-- <xacro:camera_d435 name="camera" topics_ns="camera" parent="lift_link" publish_pointcloud="true"> <origin xyz="0.02 0 0.1" rpy="0 0 0" /> </xacro:camera_d435>   -->
 <xacro:rx20_steer_wheel name="left" x_steering="-1.429" y_steering="0.404" z_steering="0.06" radius="0.150" width="0.15" flip="-1" />
 <xacro:rx20_steer_wheel name="right" x_steering="-1.429" y_steering="-0.404" z_steering="0.06" radius="0.150" width="0.15" flip="-1" />
 <xacro:rx20_front_wheel name="right" x_loading="0.0" y_loading="-0.466" z_loading="0.0" radius="0.18" width="0.18" flip="-1" />
 <xacro:rx20_front_wheel name="left" x_loading="0.0" y_loading="0.466" z_loading="0.0" radius="0.18" width="0.18" flip="-1" />
-<xacro:nav_lidar name="top"  x="0."  y="0.0" z="2" roll="0" pitch="0" yaw="0.0" resolution="1"/>
+<xacro:camera name="front"  x="0.3"  y="0" z="1.0" roll="0" pitch="0" yaw="0"/>
+<!-- <xacro:nav_lidar name="top"  x="0."  y="0.0" z="2" roll="0" pitch="0" yaw="0.0" resolution="1"/> -->
 <!-- <xacro:detection_lidar name="front"  x="0.0"  y="0.0" z="2.0" roll="0" pitch="0" yaw="0" resolution="1"/> -->
 <!-- <xacro:nav_lidar name="back"  x="-1.65"  y="0.0" z="0.0" roll="0" pitch="0" yaw="3.14509" resolution="1"/> -->

Commit message: Fixed camera frame orientation, docking possible now.

File: urdf/RX20_16/camera.xacro (robot description, xacro)
@@ -2,5 +2,5 @@
 <robot name="RX20_16" xmlns:xacro="http://www.ros.org/wiki/xacro">
 <xacro:macro name="camera" params="name x y z roll pitch yaw ">
-  <link name="${name}_camera_frame">
+  <link name="${name}_camera_link">
       <inertial>
       <origin xyz="0 0 0" rpy="0 0 0"/>
@@ -8,8 +8,8 @@
       <mass value= "0.01"/>
       </inertial>
-      <visual name="${name}_camera_frame">
+      <visual name="${name}_camera_link">
       <origin xyz="0 0 0" rpy="0 0 0"/>
       <geometry>
-       <box size="0.1 0.1 0.1"/>
+       <box size="0.1 0.05 0.05"/>
       </geometry>
       <material name="red">
@@ -20,10 +20,20 @@
   <joint name="${name}_camera_joint" type="fixed">
     <parent link="base_link" />
-    <child link="${name}_camera_frame" />
+    <child link="${name}_camera_link" />
     <origin xyz="${x} ${y} ${z}" rpy="${roll} ${pitch} ${yaw}" />
     <axis xyz="0 0 1" />
   </joint>
+  <joint name="camera_optical_joint" type="fixed">
+    <!-- these values have to be these values otherwise the gazebo camera
+        image won't be aligned properly with the frame it is supposedly
+        originating from -->
+    <origin xyz="0 0 0" rpy="-1.5708 0 -1.5708"/>
+    <parent link="${name}_camera_link"/>
+    <child link="${name}_camera_link_optical"/>
+  </joint>
+  <link name="${name}_camera_link_optical">
+  </link>
     <!-- Gazebo links and joints -->
-  <gazebo reference="${name}_camera_frame">
+  <gazebo reference="${name}_camera_link">
     <sensor name="rgbd_camera" type="rgbd_camera">
       <always_on>1</always_on>
@@ -38,5 +48,5 @@
           <far>100</far>
         </clip>
-        <optical_frame_id>${name}_camera_frame</optical_frame_id>
+        <optical_frame_id>${name}_camera_link_optical</optical_frame_id>
       </camera>
       <update_rate>10</update_rate>

File: urdf/RX20_16/main.xacro (robot description, xacro)
@@ -15,5 +15,5 @@
 <xacro:rx20_front_wheel name="right" x_loading="0.0" y_loading="-0.466" z_loading="0.0" radius="0.18" width="0.18" flip="-1" />
 <xacro:rx20_front_wheel name="left" x_loading="0.0" y_loading="0.466" z_loading="0.0" radius="0.18" width="0.18" flip="-1" />
-<xacro:camera name="front"  x="0.4"  y="0" z="0.3" roll="0" pitch="0" yaw="0"/>
+<xacro:camera name="front"  x="0.4"  y="0" z="0.3" roll="0.0" pitch="0.0" yaw="0.0"/>
 <!-- <xacro:nav_lidar name="top"  x="0."  y="0.0" z="2" roll="0" pitch="0" yaw="0.0" resolution="1"/> -->
 <!-- <xacro:detection_lidar name="front"  x="0.0"  y="0.0" z="2.0" roll="0" pitch="0" yaw="0" resolution="1"/> -->

Commit message: Attached apriltag to one end of pallet.

File: urdf/RX20_16/camera.xacro (robot description, xacro)
@@ -11,5 +11,5 @@
       <origin xyz="0 0 0" rpy="0 0 0"/>
       <geometry>
-       <box size="0.1 0.05 0.05"/>
+       <box size="0.01 0.05 0.05"/>
       </geometry>
       <material name="red">
@@ -39,11 +39,11 @@
       <always_on>1</always_on>
       <camera>
-        <horizontal_fov>1.0</horizontal_fov>
+        <horizontal_fov>1.5</horizontal_fov>
         <image>
-          <width>800</width>
-          <height>600</height>
+          <width>640</width>
+          <height>480</height>
         </image>
         <clip>
-          <near>0.3</near>
+          <near>0.03</near>
           <far>100</far>
         </clip>

File: urdf/RX20_16/main.xacro (robot description, xacro)
@@ -15,5 +15,5 @@
 <xacro:rx20_front_wheel name="right" x_loading="0.0" y_loading="-0.466" z_loading="0.0" radius="0.181" width="0.18" flip="-1" />
 <xacro:rx20_front_wheel name="left" x_loading="0.0" y_loading="0.466" z_loading="0.0" radius="0.181" width="0.18" flip="-1" />
-<xacro:camera name="front"  x="0.4"  y="0" z="0.2" roll="0.0" pitch="0.0" yaw="0.0"/>
+<xacro:camera name="front"  x="0.38"  y="0" z="-0.1" roll="0.0" pitch="0.0" yaw="0.0"/>
 <!-- <xacro:nav_lidar name="top"  x="0."  y="0.0" z="2" roll="0" pitch="0" yaw="0.0" resolution="1"/> -->
 <!-- <xacro:detection_lidar name="front"  x="0.0"  y="0.0" z="2.0" roll="0" pitch="0" yaw="0" resolution="1"/> -->
