Commit message: Forklift can move up/down manually with ros2 publish commands.

File: urdf/RX20_16/loading_forklift_joints.xacro (robot description, xacro)
@@ -47,5 +47,5 @@
   </link>
   <!-- prismatic link -->
-  <joint name="lift_joint" type="fixed">
+  <joint name="lift_joint" type="prismatic">
     <parent link="tilt_link" />
     <child link="lift_link" />
@@ -53,5 +53,5 @@
     <axis xyz="0 0 1" />
     <limit lower="-0.2" upper="2" effort="100" velocity="0.3"/>
-     <dynamics damping="100.0" friction="1"/>
+     <!-- <dynamics damping="100.0" friction="1"/> -->
   </joint>
   <link name="sideshift_link">
@@ -172,3 +172,23 @@
     <axis xyz="0 0 1" />
   </joint>
+    <!-- Gazebo plugin configuration -->
+    <ros2_control name="2DofPosition" type="system">
+        <hardware>
+            <plugin>gz_ros2_control/GazeboSimSystem</plugin>
+        </hardware>
+        <joint name="lift_joint">
+            <command_interface name="position" />
+            <command_interface name="velocity" />
+            <state_interface name="position">
+                <param name="initial_value">0.3</param>
+            </state_interface>
+            <state_interface name="velocity"/>
+            <state_interface name="effort"/>
+        </joint>
+    </ros2_control>
+    <gazebo>
+        <plugin filename="gz_ros2_control-system" name="gz_ros2_control::GazeboSimROS2ControlPlugin">
+            <parameters>$(find wb_nav2_bringup)/configs/controller.yaml</parameters>
+        </plugin>
+    </gazebo>
   </robot>

Commit message: Fork can be moved up/down with teleop keyboard.

File: urdf/RX20_16/loading_forklift_joints.xacro (robot description, xacro)
@@ -52,6 +52,6 @@
     <origin xyz="0.134 0 0.22" rpy="0 0 0" />
     <axis xyz="0 0 1" />
-    <limit lower="-0.2" upper="2" effort="100" velocity="0.3"/>
-     <!-- <dynamics damping="100.0" friction="1"/> -->
+    <limit lower="-0.149" upper="1.5" effort="100" velocity="0.3"/>
+     <dynamics damping="1.0" friction="0.001"/>
   </joint>
   <link name="sideshift_link">
@@ -79,5 +79,5 @@
     <origin xyz="0.06 0 -0.25" rpy="0 0 0" />
     <axis xyz="0 1 0" />
-    <limit lower="-0.2" upper="0.2" effort="100" velocity="0.3"/>
+    <limit lower="-0.15" upper="0.2" effort="100" velocity="0.3"/>
      <dynamics damping="10" friction="1"/>
   </joint>

Commit message: Move forks further apart to make pallet docking easier.

File: urdf/RX20_16/loading_forklift_joints.xacro (robot description, xacro)
@@ -63,5 +63,5 @@
     <collision >
     <origin xyz="0 0 0" rpy="0 0 0"/>
-    <geometry> <mesh filename="file:$(find wb_nav2_bringup)/urdf/RX20_16/meshes/sideshift_link.dae" />
+    <geometry> <mesh filename="file:$(find wb_nav2_bringup)/urdf/RX20_16/meshes/sideshift_link_wide.dae" />
     </geometry>
     </collision>
@@ -69,5 +69,5 @@
     <origin xyz="0 0 0" rpy="0 0 0"/>
     <geometry>
-          <mesh filename="file:$(find wb_nav2_bringup)/urdf/RX20_16/meshes/sideshift_link.dae" />
+          <mesh filename="file:$(find wb_nav2_bringup)/urdf/RX20_16/meshes/sideshift_link_wide.dae" />
     </geometry>
     </visual>

Commit message: Added mid-width fork. Fixed fork collision model.

File: urdf/RX20_16/loading_forklift_joints.xacro (robot description, xacro)
@@ -52,5 +52,5 @@
     <origin xyz="0.134 0 0.22" rpy="0 0 0" />
     <axis xyz="0 0 1" />
-    <limit lower="-0.149" upper="1.5" effort="100" velocity="0.3"/>
+    <limit lower="-0.25" upper="1.5" effort="100" velocity="0.3"/>
      <dynamics damping="1.0" friction="0.001"/>
   </joint>
@@ -63,5 +63,6 @@
     <collision >
     <origin xyz="0 0 0" rpy="0 0 0"/>
-    <geometry> <mesh filename="file:$(find wb_nav2_bringup)/urdf/RX20_16/meshes/sideshift_link_wide.dae" />
+    <geometry>
+      <mesh filename="file:$(find wb_nav2_bringup)/urdf/RX20_16/meshes/sideshift_link_mid_short.dae" />
     </geometry>
     </collision>
@@ -69,54 +70,17 @@
     <origin xyz="0 0 0" rpy="0 0 0"/>
     <geometry>
-          <mesh filename="file:$(find wb_nav2_bringup)/urdf/RX20_16/meshes/sideshift_link_wide.dae" />
+      <mesh filename="file:$(find wb_nav2_bringup)/urdf/RX20_16/meshes/sideshift_link_mid_short.dae" />
     </geometry>
     </visual>
   </link>
-  <!-- prismatic link -->
   <joint name="sideshift_joint" type="fixed">
     <parent link="lift_link" />
     <child link="sideshift_link" />
-    <origin xyz="0.06 0 -0.25" rpy="0 0 0" />
+    <origin xyz="0.06 0 -0.20" rpy="0 0 0" />
     <axis xyz="0 1 0" />
     <limit lower="-0.15" upper="0.2" effort="100" velocity="0.3"/>
      <dynamics damping="10" friction="1"/>
   </joint>
-  <!-- <transmission name="tran1">
-    <type>transmission_interface/SimpleTransmission</type>
-    <joint name="tilt_joint">
-      <hardwareInterface>hardware_interface/EffortJointInterface</hardwareInterface>
-    </joint>
-    <actuator name="motor1">
-      <hardwareInterface>hardware_interface/EffortJointInterface</hardwareInterface>
-      <mechanicalReduction>1</mechanicalReduction>
-    </actuator>
-  </transmission>
-  <transmission name="tran2">
-    <type>transmission_interface/SimpleTransmission</type>
-    <joint name="lift_joint">
-      <hardwareInterface>hardware_interface/EffortJointInterface</hardwareInterface>
-    </joint>
-    <actuator name="motor2">
-      <hardwareInterface>hardware_interface/EffortJointInterface</hardwareInterface>
-      <mechanicalReduction>1</mechanicalReduction>
-    </actuator>
-  </transmission>
-  <transmission name="tran3">
-    <type>transmission_interface/SimpleTransmission</type>
-    <joint name="sideshift_joint">
-      <hardwareInterface>hardware_interface/EffortJointInterface</hardwareInterface>
-    </joint>
-    <actuator name="motor3">
-      <hardwareInterface>hardware_interface/EffortJointInterface</hardwareInterface>
-      <mechanicalReduction>1</mechanicalReduction>
-    </actuator>
-  </transmission> -->
-  <!-- <gazebo>
-    <plugin name="gazebo_ros_control" filename="libgazebo_ros_control.so">
-      <robotNamespace>/RX20_16</robotNamespace>
-      <robotSimType>gazebo_ros_control/DefaultRobotHWSim</robotSimType>
-    </plugin>
-  </gazebo> -->
-  <link name='box1'>
+   <!-- <link name='box1'>
     <collision>
       <geometry>
@@ -124,9 +88,9 @@
       </geometry>
     </collision>
-    <!-- <visual>
+    <visual>
       <geometry>
         <box size="0.8 0.08 0.04"/>
       </geometry>
-    </visual> -->
+    </visual>
   </link>
   <joint name="pad_joint1" type="fixed">
@@ -142,9 +106,9 @@
       </geometry>
     </collision>
-    <!-- <visual>
+    <visual>
       <geometry>
         <box size="0.8 0.08 0.04"/>
       </geometry>
-    </visual> -->
+    </visual>
   </link>
   <joint name="pad_joint2" type="fixed">
@@ -160,9 +124,9 @@
       </geometry>
     </collision>
-    <!-- <visual>
+    <visual>
       <geometry>
         <box size="0.02 0.2 0.1"/>
       </geometry>
-    </visual> -->
+    </visual>
   </link>
   <joint name="pad_joint" type="fixed">
@@ -171,5 +135,5 @@
     <origin xyz="0.0 0.0 0.05" rpy="0 0 0" />
     <axis xyz="0 0 1" />
-  </joint>
+  </joint> -->
     <!-- Gazebo plugin configuration -->
     <ros2_control name="2DofPosition" type="system">
@@ -181,5 +145,5 @@
             <command_interface name="velocity" />
             <state_interface name="position">
-                <param name="initial_value">-0.1</param>
+                <param name="initial_value">-0.15</param>
             </state_interface>
             <state_interface name="velocity"/>

Commit message: Darkened fork so it is easier to see.

File: urdf/RX20_16/loading_forklift_joints.xacro (robot description, xacro)
@@ -64,5 +64,5 @@
     <origin xyz="0 0 0" rpy="0 0 0"/>
     <geometry>
-      <mesh filename="file:$(find wb_nav2_bringup)/urdf/RX20_16/meshes/sideshift_link_mid_short.dae" />
+      <mesh filename="file:$(find wb_nav2_bringup)/urdf/RX20_16/meshes/sideshift_link_mid_short_dark.dae" />
     </geometry>
     </collision>
@@ -70,5 +70,5 @@
     <origin xyz="0 0 0" rpy="0 0 0"/>
     <geometry>
-      <mesh filename="file:$(find wb_nav2_bringup)/urdf/RX20_16/meshes/sideshift_link_mid_short.dae" />
+      <mesh filename="file:$(find wb_nav2_bringup)/urdf/RX20_16/meshes/sideshift_link_mid_short_dark.dae" />
     </geometry>
     </visual>
